Commit message: Can run launch file and rviz pops up with a sphere

File: turtle_brick/urdf/turtle.urdf.xacro (robot description, xacro)
@@ -1,5 +1,5 @@
 <?xml version="1.0"?>
-<robot name="myfirst">
-  <link name="base_link">
+<robot name="turtle_robot">
+  <link name="base">
     <visual>
       <geometry>

Commit message: Added all four frame, not all static either

File: turtle_brick/urdf/turtle.urdf.xacro (robot description, xacro)
@@ -1,5 +1,5 @@
 <?xml version="1.0"?>
 <robot name="turtle_robot">
-  <link name="base">
+  <link name="base_link">
     <visual>
       <geometry>

Commit message: URDF looking done

File: turtle_brick/urdf/turtle.urdf.xacro (robot description, xacro)
@@ -1,10 +1,32 @@
 <?xml version="1.0"?>
 <robot name="turtle_robot">
-  <link name="base_link">
+  <link name="wheel">
     <visual>
       <geometry>
-        <sphere radius="0.2"/>
+        <cylinder length="0.1" radius="0.2"/>
       </geometry>
     </visual>
   </link>
+  <link name="stem">
+    <visual>
+      <geometry>
+        <cylinder length="0.5" radius="0.05"/>
+      </geometry>
+    </visual>
+  </link>
+  <joint name="wheel_to_stem" type="fixed">
+    <parent link="wheel"/>
+    <child link="stem"/>
+  </joint>
+  <link name="platform">
+    <visual>
+      <geometry>
+        <cylinder length="0.025" radius="0.3"/>
+      </geometry>
+    </visual>
+  </link>
+  <joint name="stem_to_platform" type="fixed">
+    <parent link="stem"/>
+    <child link="platform"/>
+  </joint>
 </robot>

Commit message: Joints and urdf looking good. Still need to add xacro though

File: turtle_brick/urdf/turtle.urdf.xacro (robot description, xacro)
@@ -1,4 +1,23 @@
 <?xml version="1.0"?>
-<robot name="turtle_robot">
+<robot xmlns:xacro="http://www.ros.org/wiki/xacro" name="turtle_robot">
+  <link name="base_link">
+    <visual>
+      <geometry>
+        <box size="0.3 0.3 0.3"/>
+      </geometry>
+    </visual>
+  </link>
+  <link name="stem">
+    <visual>
+      <geometry>
+        <cylinder length="0.2" radius="0.05"/>
+      </geometry>
+    </visual>
+  </link>
+  <joint name="base_to_stem" type="fixed">
+    <parent link="base_link"/>
+    <child link="stem"/>
+    <origin rpy="0 0 0" xyz="0 0 -0.15"/>
+  </joint>
   <link name="wheel">
     <visual>
@@ -8,14 +27,26 @@
     </visual>
   </link>
-  <link name="stem">
+  <joint name="spin_wheel" type="continuous">
+    <axis xyz="0 0 1"/>
+    <parent link="stem"/>
+    <child link="wheel"/>
+    <origin rpy="0 1.57 0" xyz="0 0 -0.3"/>
+  </joint>
+  <joint name="turn_wheel" type="continuous">
+    <parent link="stem"/>
+    <child link="wheel"/>
+    <origin rpy="0 1.57 0" xyz="0 0 -0.3"/>
+  </joint>
+  <link name="tube">
     <visual>
       <geometry>
-        <cylinder length="0.5" radius="0.05"/>
+        <cylinder length="0.4" radius="0.05"/>
       </geometry>
     </visual>
   </link>
-  <joint name="wheel_to_stem" type="fixed">
-    <parent link="wheel"/>
-    <child link="stem"/>
+  <joint name="base_to_tube" type="fixed">
+    <parent link="base_link"/>
+    <child link="tube"/>
+    <origin xyz="0 0 0.3"/>
   </joint>
   <link name="platform">
@@ -26,7 +57,10 @@
     </visual>
   </link>
-  <joint name="stem_to_platform" type="fixed">
-    <parent link="stem"/>
+  <joint name="tilt_platform" type="revolute">
+    <parent link="tube"/>
     <child link="platform"/>
+    <origin xyz="0 0 0.2"/>
+    <axis xyz="0 1 0"/>
+    <limit effort="1000.0" lower="-1.570" upper="1.57" velocity="0.5"/>
   </joint>
 </robot>

Commit message: Fixed joint axes

File: turtle_brick/urdf/turtle.urdf.xacro (robot description, xacro)
@@ -15,8 +15,9 @@
     </visual>
   </link>
-  <joint name="base_to_stem" type="fixed">
+  <joint name="turn_wheel" type="continuous">
+    <axis xyz="0 0 1"/>
     <parent link="base_link"/>
     <child link="stem"/>
-    <origin rpy="0 0 0" xyz="0 0 -0.15"/>
+    <origin xyz="0 0 -0.15"/>
   </joint>
   <link name="wheel">
@@ -29,9 +30,4 @@
   <joint name="spin_wheel" type="continuous">
     <axis xyz="0 0 1"/>
-    <parent link="stem"/>
-    <child link="wheel"/>
-    <origin rpy="0 1.57 0" xyz="0 0 -0.3"/>
-  </joint>
-  <joint name="turn_wheel" type="continuous">
     <parent link="stem"/>
     <child link="wheel"/>

Commit message: Turtle mvoes!

File: turtle_brick/urdf/turtle.urdf.xacro (robot description, xacro)
@@ -26,4 +26,5 @@
         <cylinder length="0.1" radius="0.2"/>
       </geometry>
+      <origin rpy="1.57 0 0 "/>
     </visual>
   </link>

Commit message: Imported yaml and set up xacro.

File: turtle_brick/urdf/turtle.urdf.xacro (robot description, xacro)
@@ -1,4 +1,8 @@
 <?xml version="1.0"?>
 <robot xmlns:xacro="http://www.ros.org/wiki/xacro" name="turtle_robot">
+<xacro:property name="yaml_file" value="$(find package)/config/turtle.yaml" />
+<xacro:property name="props" value="${load_yaml(yaml_file)}"/>
+<xacro:property name="platform_height" value="0.4" />
+<xacro:property name="wheel_radius" value="0.2" />
   <link name="base_link">
     <visual>
@@ -24,7 +28,7 @@
     <visual>
       <geometry>
-        <cylinder length="0.1" radius="0.2"/>
+        <cylinder length="0.1" radius="${wheel_radius}"/>
       </geometry>
-      <origin rpy="1.57 0 0 "/>
+      <origin rpy="${pi/2} 0 0 "/>
     </visual>
   </link>
@@ -33,10 +37,10 @@
     <parent link="stem"/>
     <child link="wheel"/>
-    <origin rpy="0 1.57 0" xyz="0 0 -0.3"/>
+    <origin rpy="0 ${pi/2} 0" xyz="0 0 -0.3"/>
   </joint>
   <link name="tube">
     <visual>
       <geometry>
-        <cylinder length="0.4" radius="0.05"/>
+        <cylinder length="${platform_height}" radius="0.05"/>
       </geometry>
     </visual>
@@ -57,7 +61,7 @@
     <parent link="tube"/>
     <child link="platform"/>
-    <origin xyz="0 0 0.2"/>
+    <origin xyz="0 0 ${platform_height/2 + 0.025/2}"/>
     <axis xyz="0 1 0"/>
-    <limit effort="1000.0" lower="-1.570" upper="1.57" velocity="0.5"/>
+    <limit effort="1000.0" lower="${-pi/2}" upper="${pi/2}" velocity="0.5"/>
   </joint>
 </robot>

Commit message: yaml updated. Nodes not crashing anymore!

File: turtle_brick/urdf/turtle.urdf.xacro (robot description, xacro)
@@ -1,8 +1,10 @@
 <?xml version="1.0"?>
 <robot xmlns:xacro="http://www.ros.org/wiki/xacro" name="turtle_robot">
-<xacro:property name="yaml_file" value="$(find package)/config/turtle.yaml" />
+<xacro:property name="yaml_file" value="$(find turtle_brick)/turtle.yaml" />
 <xacro:property name="props" value="${load_yaml(yaml_file)}"/>
-<xacro:property name="platform_height" value="0.4" />
-<xacro:property name="wheel_radius" value="0.2" />
+<xacro:property name="star" value="${props['/**']}" />
+<xacro:property name="ros_parameters" value="${star['ros__parameters']}" />
+<xacro:property name="wheel_radius" value="${ros_parameters['wheel_radius']}" />
+<xacro:property name="platform_height" value="${ros_parameters['platform_height']}" />
   <link name="base_link">
     <visual>

Commit message: Fixed yaml loading bug

File: turtle_brick/urdf/turtle.urdf.xacro (robot description, xacro)
@@ -7,4 +7,5 @@
 <xacro:property name="wheel_radius" value="${ros_parameters['wheel_radius']}" />
 <xacro:property name="platform_height" value="${ros_parameters['platform_height']}" />
+<xacro:property name="tube_length" value="${platform_height - 0.025 - 0.2 - 0.3 - wheel_radius*2}" />
   <link name="base_link">
     <visual>
@@ -25,5 +26,5 @@
     <parent link="base_link"/>
     <child link="stem"/>
-    <origin xyz="0 0 -0.15"/>
+    <origin xyz="0 0 -0.25"/>
   </joint>
   <link name="wheel">
@@ -39,10 +40,10 @@
     <parent link="stem"/>
     <child link="wheel"/>
-    <origin rpy="0 ${pi/2} 0" xyz="0 0 -0.3"/>
+    <origin rpy="0 ${pi/2} 0" xyz="0 0 -${0.1+wheel_radius}"/>
   </joint>
   <link name="tube">
     <visual>
       <geometry>
-        <cylinder length="${platform_height}" radius="0.05"/>
+        <cylinder length="${tube_length}" radius="0.05"/>
       </geometry>
     </visual>
@@ -51,5 +52,5 @@
     <parent link="base_link"/>
     <child link="tube"/>
-    <origin xyz="0 0 0.3"/>
+    <origin xyz="0 0 ${0.15 + 0.5*tube_length}"/>
   </joint>
   <link name="platform">
@@ -63,5 +64,5 @@
     <parent link="tube"/>
     <child link="platform"/>
-    <origin xyz="0 0 ${platform_height/2 + 0.025/2}"/>
+    <origin xyz="0 0 ${tube_length/2 + 0.025/2}"/>
     <axis xyz="0 1 0"/>
     <limit effort="1000.0" lower="${-pi/2}" upper="${pi/2}" velocity="0.5"/>

Commit message: Changed urdf to make stem variable instead of tube

File: turtle_brick/urdf/turtle.urdf.xacro (robot description, xacro)
@@ -7,5 +7,5 @@
 <xacro:property name="wheel_radius" value="${ros_parameters['wheel_radius']}" />
 <xacro:property name="platform_height" value="${ros_parameters['platform_height']}" />
-<xacro:property name="tube_length" value="${platform_height - 0.025 - 0.2 - 0.3 - wheel_radius*2}" />
+<xacro:property name="stem_length" value="${platform_height - 0.025 - 0.3 - 0.3 - wheel_radius*2}" />
   <link name="base_link">
     <visual>
@@ -18,5 +18,5 @@
     <visual>
       <geometry>
-        <cylinder length="0.2" radius="0.05"/>
+        <cylinder length="${stem_length}" radius="0.05"/>
       </geometry>
     </visual>
@@ -26,5 +26,5 @@
     <parent link="base_link"/>
     <child link="stem"/>
-    <origin xyz="0 0 -0.25"/>
+    <origin xyz="0 0 -${0.15+stem_length/2}"/>
   </joint>
   <link name="wheel">
@@ -40,10 +40,10 @@
     <parent link="stem"/>
     <child link="wheel"/>
-    <origin rpy="0 ${pi/2} 0" xyz="0 0 -${0.1+wheel_radius}"/>
+    <origin rpy="0 ${pi/2} 0" xyz="0 0 -${stem_length/2+wheel_radius}"/>
   </joint>
   <link name="tube">
     <visual>
       <geometry>
-        <cylinder length="${tube_length}" radius="0.05"/>
+        <cylinder length="0.3" radius="0.05"/>
       </geometry>
     </visual>
@@ -52,5 +52,5 @@
     <parent link="base_link"/>
     <child link="tube"/>
-    <origin xyz="0 0 ${0.15 + 0.5*tube_length}"/>
+    <origin xyz="0 0 ${0.15 + 0.5*0.3}"/>
   </joint>
   <link name="platform">
@@ -64,5 +64,5 @@
     <parent link="tube"/>
     <child link="platform"/>
-    <origin xyz="0 0 ${tube_length/2 + 0.025/2}"/>
+    <origin xyz="0 0 ${0.3/2 + 0.025/2}"/>
     <axis xyz="0 1 0"/>
     <limit effort="1000.0" lower="${-pi/2}" upper="${pi/2}" velocity="0.5"/>

Commit message: Wheel spinning

File: turtle_brick/urdf/turtle.urdf.xacro (robot description, xacro)
@@ -37,5 +37,5 @@
   </link>
   <joint name="spin_wheel" type="continuous">
-    <axis xyz="0 0 1"/>
+    <axis xyz="0 1 0"/>
     <parent link="stem"/>
     <child link="wheel"/>
